File: NU25 Connector Pinout/PCB/NU25 Connector Pinout/NU25 Connector Pinout.kicad_sch (KiCad schematic)
At the start: 252 parts, among them J1 Conn_01x01_Pin, J10 Conn_01x01_Pin, J100 Conn_01x01_Pin, J101 Conn_01x01_Pin, J102 Conn_01x01_Pin, J103 Conn_01x01_Pin, J104 Conn_01x01_Pin, J105 Conn_01x01_Pin, J106 Conn_01x01_Pin, J107 Conn_01x01_Pin, J108 Conn_01x01_Pin, J109 Conn_01x01_Pin, J11 Conn_01x01_Pin, J110 Conn_01x01_Pin, J111 Conn_01x01_Pin, J112 Conn_01x01_Pin, J113 Conn_01x01_Pin, J114 Conn_01x01_Pin, J115 Conn_01x01_Pin, J116 Conn_01x01_Pin, J117 Conn_01x01_Pin, J118 Conn_01x01_Pin, J119 Conn_01x01_Pin, J12 Conn_01x01_Pin, J120 Conn_01x01_Pin, J121 Conn_01x01_Pin, J122 Conn_01x01_Pin, J123 Conn_01x01_Pin, J124 Conn_01x01_Pin, J125 Conn_01x01_Pin, J126 Conn_01x01_Pin, J127 Conn_01x01_Pin, J128 Conn_01x01_Pin, J129 Conn_01x01_Pin, J13 Conn_01x01_Pin, J130 Conn_01x01_Pin, J131 Conn_01x01_Pin, J132 Conn_01x01_Pin, J133 Conn_01x01_Pin, J134 Conn_01x01_Pin, J135 Conn_01x01_Pin, J136 Conn_01x01_Pin, J137 Conn_01x01_Pin, J138 Conn_01x01_Pin, J139 Conn_01x01_Pin, J14 Conn_01x01_Pin, J140 Conn_01x01_Pin, J141 Conn_01x01_Pin, J142 Conn_01x01_Pin, J143 Conn_01x01_Pin, J144 Conn_01x01_Pin, J145 Conn_01x01_Pin, J146 Conn_01x01_Pin, J147 Conn_01x01_Pin, J148 Conn_01x01_Pin, J149 Conn_01x01_Pin, J15 Conn_01x01_Pin, J150 Conn_01x01_Pin, J151 Conn_01x01_Pin, J152 Conn_01x01_Pin, J153 Conn_01x01_Pin, J154 Conn_01x01_Pin, J155 Conn_01x01_Pin, J156 Conn_01x01_Pin, J157 Conn_01x01_Pin, J158 Conn_01x01_Pin, J159 Conn_01x01_Pin, J16 Conn_01x01_Pin, J160 Conn_01x01_Pin, J161 Conn_01x01_Pin, J162 Conn_01x01_Pin, J163 Conn_01x01_Pin, J164 Conn_01x01_Pin, J165 Conn_01x01_Pin, J166 Conn_01x01_Pin, J167 Conn_01x01_Pin, J168 Conn_01x01_Pin, J169 Conn_01x01_Pin, J17 Conn_01x01_Pin, J170 Conn_01x01_Pin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

Commit message: hv connectors, nu25 connector pinout schematic
ordered the hv connectors into files for where they will go

continued work on the nu25 schematic
Parts:
- added J253, J254, J255, J256, J257, J258, J259, J260, J261, J262, J263, J264, J265, J266, J267, J268, J269, J270, J271, J272, J273, J274, J275, J276, J277, J278, J279, J280, J281, J282, J283, J284, J285, J286, J287, J288, J289, J290, J291, J292, J293, J294, J295, J296, J297, J298, J299, J300, J301, J302, J303, J304, J305, J306, J307, J308, J309, J310, J311, J312, J313, J314, J315, J316, J317, J318, J319, J320, J321, J322, J323, J324, J325, J326, J327, J328, J329, J330, J331, J332, J333, J334, J335, J336, J337, J338, J339, J340, J341, J342, J343, J344, J345, J346, J347, J348, J349, J350, J351, J352, J353, J354, J355, J356, J357, J358, J359, J360, J361, J362, J363, J364, J365, J366, J367, J368, J369, J370, J371, J372, J373, J374, J375, J376, J377, J378, J379, J380, J381, J382, J383, J384, J385, J386, J387, J388, J389, J390, J391, J392, J393, J394, J395, J396, J397, J398, J399, J400, J401, J402, J403, J404, J405, J406, J407, J408, J409, J410, J411, J412, J413, J414, J415, J416, J417, J418, J419, J420, J421, J422, J423, J424, J425, J426, J427, J428, J429, J430, J431, J432, J433, J434, J435, J436, J437, J438, J439, J440, J441, J442, J443, J444, J445, J446, J447, J448, J449, J450, J451, J452, J453, J454, J455, J456, J457, J458, J459, J460, J461, J462, J463, J464, J465, J466, J467, J468, J469, J470, J471, J472, J473, J474, J475, J476, J477, J478, J479, J480, J481, J482, J483, J484, J485, J486, J487, J488, J489, J490, J491, J492, J493, J494, J495, J496, J497, J498, J499, J500, J501, J502, J503, J504, J505, J506, J507, J508, J509, J510, J511, J512, J513, J514, J515, J516, J517, J518, J519, J520, J521, J522, J523, J524, J525, J526, J527, J528, J529, J530, J531, J532, J533, J534, J535, J536, J537, J538, J539, J540, J541, J542, J543, J544, J545, J546, J547, J548, J549, J550, J551, J552, J553, J554, J555, J556, J557, J558, J559, J560, J561, J562, J563, J564, J565, J566, J567, J568, J569, J570, J571, J572, J573, J574, J575, J576, J577, J578, J579, J580, J581, J582, J583, J584, J585, J586, J587, J588, J589, J590, J591, J592, J593, J594, J595, J596, J597, J598, J599, J600, J601, J602, J603, J604, J605, J606, J607, J608, J609, J610, J611, J612, J613, J614, J615, J616, J617, J618, J619, J620, J621, J622, J623, J624, J625, J626, J627, J628, J629, J630, J631, J632, J633, J634, J635, J636, J637, J638, J639, J640, J641, J642, J643, J644, J645, J646, J647, J648, J649, J650, J651, J652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: Conn_01x01_Pin, symbol Connector:Conn_01x01_Pin
Connections:
- net at J14. (Pin_1): now also J20. (Pin_1)
- net at J22. (Pin_1): now also J5. (Pin_1)
- net at J118. (Pin_1): now also J115. (Pin_1)
- net at J219. (Pin_1): now also J171. (Pin_1)
- net at J90. (Pin_1): now also J130. (Pin_1); no longer J140. (Pin_1)
- net at J58. (Pin_1): now also J137. (Pin_1)
- net at J122. (Pin_1): now also J409. (Pin_1)
- net at J27. (Pin_1): now also J16. (Pin_1)
- net at J128. (Pin_1): now also J103. (Pin_1)
- net at J246. (Pin_1): now also J405. (Pin_1)
- net at J19. (Pin_1): now also J15. (Pin_1)
- net at J194. (Pin_1): now also J240. (Pin_1)
- net at J175. (Pin_1): now also J229. (Pin_1)
- net at J191. (Pin_1): now also J237. (Pin_1)
- net at J241. (Pin_1): now also J195. (Pin_1)
- net at J234. (Pin_1): now also J188. (Pin_1)
- net at J125. (Pin_1): now also J102. (Pin_1)
- net at J214. (Pin_1): now also J166. (Pin_1)
- net at J76. (Pin_1): now also J135. (Pin_1)
- net at J245. (Pin_1): now also J406. (Pin_1)
- net at J170. (Pin_1): now also J218. (Pin_1)
- net at J174. (Pin_1): now also J228. (Pin_1)
- net at J123. (Pin_1): now also J112. (Pin_1)
- net at J63. (Pin_1): now also J133. (Pin_1)
- net at J167. (Pin_1): now also J215. (Pin_1)
- net at J28. (Pin_1): now also J8. (Pin_1)
- net at J9. (Pin_1): now also J21. (Pin_1)
- net at J6. (Pin_1): now also J11. (Pin_1)
- net at J136. (Pin_1): now also J81. (Pin_1)
- net at J187. (Pin_1): now also J233. (Pin_1)
- net at J168. (Pin_1): now also J216. (Pin_1)
- net at J163. (Pin_1): now also J349. (Pin_1)
- net at J250. (Pin_1): now also J401. (Pin_1); no longer J164. (Pin_1)
- net at J186. (Pin_1): now also J232. (Pin_1)
- net at J32. (Pin_1): now also J31. (Pin_1)
- net at J158. (Pin_1): now also J346. (Pin_1)
- net at J57. (Pin_1): now also J138. (Pin_1)
- net at J190. (Pin_1): now also J236. (Pin_1)
- net at J30. (Pin_1): now also J29. (Pin_1)
- net at J244. (Pin_1): now also J407. (Pin_1)
- net at J129. (Pin_1): now also J89. (Pin_1)
- net at J157. (Pin_1): now also J339. (Pin_1)
- net at J116. (Pin_1): now also J113. (Pin_1)
- net at J17. (Pin_1): now also J24. (Pin_1)
- net at J127. (Pin_1): now also J105. (Pin_1)
- net at J173. (Pin_1): now also J227. (Pin_1)
- net at J183. (Pin_1): now also J178. (Pin_1), J179. (Pin_1), J182. (Pin_1), J184. (Pin_1), J318. (Pin_1), J712. (Pin_1)
- net at J243. (Pin_1): now also J408. (Pin_1)
- net at J192. (Pin_1): now also J238. (Pin_1)
- net at J180. (Pin_1): now also J321. (Pin_1)
- net at J176. (Pin_1): now also J230. (Pin_1)
- net at J239. (Pin_1): now also J193. (Pin_1)
- net at J10. (Pin_1): now also J18. (Pin_1)
- net at J74. (Pin_1): now also J132. (Pin_1)
- net at J211. (Pin_1): now also J331. (Pin_1)
- net at J208. (Pin_1): now also J323. (Pin_1)
- net at J12. (Pin_1): now also J23. (Pin_1)
- net at J101. (Pin_1): now also J126. (Pin_1)
- net at J114. (Pin_1): now also J117. (Pin_1)
- net at J66. (Pin_1): now also J140. (Pin_1)
- net at J109. (Pin_1): now also J124. (Pin_1)
- net at J26. (Pin_1): now also J13. (Pin_1)
- net at J235. (Pin_1): now also J189. (Pin_1)
- net at J159. (Pin_1): now also J348. (Pin_1)
- net at J25. (Pin_1): now also J7. (Pin_1)
- net at J162. (Pin_1): now also J347. (Pin_1)
- net at J248. (Pin_1): now also J403. (Pin_1)
- net at J139. (Pin_1): now also J67. (Pin_1)
- net at J220. (Pin_1): now also J172. (Pin_1)
- net at J217. (Pin_1): now also J169. (Pin_1)
- net at J206. (Pin_1): now also J325. (Pin_1)
- net at J120. (Pin_1): now also J411. (Pin_1)
- net at J181. (Pin_1): now also J322. (Pin_1)
- net at J121. (Pin_1): now also J410. (Pin_1)
- net at J207. (Pin_1): now also J328. (Pin_1)
- net at J196. (Pin_1): now also J242. (Pin_1)
- net at J161. (Pin_1): now also J338. (Pin_1)
- net at J210. (Pin_1): now also J335. (Pin_1)
- net at J247. (Pin_1): now also J404. (Pin_1)
- net at J209. (Pin_1): now also J327. (Pin_1)
- net at J252. (Pin_1): now also J308. (Pin_1)
- net at J249. (Pin_1): now also J402. (Pin_1)
- net at J131. (Pin_1): now also J75. (Pin_1)
- net at J251. (Pin_1): now also J307. (Pin_1)
- net at J177. (Pin_1): now also J319. (Pin_1)
- net at J205. (Pin_1): now also J324. (Pin_1)
- net at J160. (Pin_1): now also J340. (Pin_1)
- net at J119. (Pin_1): now also J412. (Pin_1)
- net at J212. (Pin_1): now also J329. (Pin_1), J332. (Pin_1)
- new net: J354. (Pin_1), J392. (Pin_1)
- new net: J575. (Pin_1), J607. (Pin_1)
- new net: J508. (Pin_1), J554. (Pin_1)
- new net: J345. (Pin_1), J397. (Pin_1)
- new net: J442. (Pin_1), J463. (Pin_1)
- new net: J584. (Pin_1), J616. (Pin_1)
- new net: J428. (Pin_1), J476. (Pin_1)
- new net: J492. (Pin_1), J570. (Pin_1)
- new net: J591. (Pin_1), J623. (Pin_1)
- new net: J429. (Pin_1), J475. (Pin_1)
- new net: J359. (Pin_1), J387. (Pin_1)
- new net: J497. (Pin_1), J565. (Pin_1)
- new net: J528. (Pin_1), J535. (Pin_1)
- new net: J311. (Pin_1), J312. (Pin_1), J313. (Pin_1), J315. (Pin_1), J316. (Pin_1), J317. (Pin_1), J711. (Pin_1)
- new net: J494. (Pin_1), J568. (Pin_1)
- new net: J531. (Pin_1), J532. (Pin_1)
- new net: J502. (Pin_1), J560. (Pin_1)
- new net: J256. (Pin_1), J310. (Pin_1)
- new net: J449. (Pin_1), J456. (Pin_1)
- new net: J513. (Pin_1), J549. (Pin_1)
- new net: J523. (Pin_1), J540. (Pin_1)
- new net: J451. (Pin_1), J454. (Pin_1)
- new net: J505. (Pin_1), J557. (Pin_1)
- new net: J585. (Pin_1), J617. (Pin_1)
- new net: J351. (Pin_1), J395. (Pin_1)
- new net: J420. (Pin_1), J484. (Pin_1)
- new net: J511. (Pin_1), J551. (Pin_1)
- new net: J595. (Pin_1), J627. (Pin_1)
- new net: J498. (Pin_1), J564. (Pin_1)
- new net: J448. (Pin_1), J457. (Pin_1)
- new net: J601. (Pin_1), J633. (Pin_1)
- new net: J363. (Pin_1), J384. (Pin_1)
- new net: J416. (Pin_1), J488. (Pin_1)
- new net: J587. (Pin_1), J619. (Pin_1)
- new net: J352. (Pin_1), J394. (Pin_1)
- new net: J436. (Pin_1), J468. (Pin_1)
- new net: J571. (Pin_1), J603. (Pin_1)
- new net: J598. (Pin_1), J630. (Pin_1)
- new net: J602. (Pin_1), J634. (Pin_1)
- new net: J506. (Pin_1), J556. (Pin_1)
- new net: J357. (Pin_1), J389. (Pin_1)
- new net: J576. (Pin_1), J608. (Pin_1)
- new net: J431. (Pin_1), J473. (Pin_1)
- new net: J356. (Pin_1), J390. (Pin_1)
- new net: J495. (Pin_1), J567. (Pin_1)
- new net: J421. (Pin_1), J483. (Pin_1)
- new net: J597. (Pin_1), J629. (Pin_1)
- new net: J509. (Pin_1), J553. (Pin_1)
- new net: J440. (Pin_1), J465. (Pin_1)
- new net: J450. (Pin_1), J455. (Pin_1)
- new net: J493. (Pin_1), J569. (Pin_1)
- new net: J577. (Pin_1), J609. (Pin_1)
- new net: J438. (Pin_1), J466. (Pin_1)
- new net: J592. (Pin_1), J624. (Pin_1)
- new net: J512. (Pin_1), J550. (Pin_1)
- new net: J522. (Pin_1), J541. (Pin_1)
- new net: J369. (Pin_1), J378. (Pin_1)
- new net: J504. (Pin_1), J558. (Pin_1)
- new net: J596. (Pin_1), J628. (Pin_1)
- new net: J588. (Pin_1), J620. (Pin_1)
- new net: J443. (Pin_1), J462. (Pin_1)
- new net: J432. (Pin_1), J472. (Pin_1)
- new net: J365. (Pin_1), J382. (Pin_1)
- new net: J500. (Pin_1), J562. (Pin_1)
- new net: J364. (Pin_1), J383. (Pin_1)
- new net: J355. (Pin_1), J391. (Pin_1)
- new net: J529. (Pin_1), J534. (Pin_1)
- new net: J510. (Pin_1), J552. (Pin_1)
- new net: J520. (Pin_1), J543. (Pin_1)
- new net: J446. (Pin_1), J459. (Pin_1)
- new net: J430. (Pin_1), J474. (Pin_1)
- new net: J572. (Pin_1), J604. (Pin_1)
- new net: J589. (Pin_1), J621. (Pin_1)
- new net: J525. (Pin_1), J538. (Pin_1)
- new net: J358. (Pin_1), J388. (Pin_1)
- new net: J583. (Pin_1), J615. (Pin_1)
- new net: J519. (Pin_1), J544. (Pin_1)
- new net: J344. (Pin_1), J398. (Pin_1)
- new net: J574. (Pin_1), J606. (Pin_1)
- new net: J330. (Pin_1), J334. (Pin_1)
- new net: J371. (Pin_1), J376. (Pin_1)
- new net: J445. (Pin_1), J460. (Pin_1)
- new net: J425. (Pin_1), J479. (Pin_1)
- new net: J593. (Pin_1), J625. (Pin_1)
- new net: J417. (Pin_1), J487. (Pin_1)
- new net: J433. (Pin_1), J471. (Pin_1)
- new net: J368. (Pin_1), J379. (Pin_1)
- new net: J521. (Pin_1), J542. (Pin_1)
- new net: J586. (Pin_1), J618. (Pin_1)
- new net: J413. (Pin_1), J491. (Pin_1)
- new net: J496. (Pin_1), J566. (Pin_1)
- new net: J441. (Pin_1), J464. (Pin_1)
- new net: J515. (Pin_1), J547. (Pin_1)
- new net: J361. (Pin_1), J386. (Pin_1)
- new net: J600. (Pin_1), J632. (Pin_1)
- new net: J594. (Pin_1), J626. (Pin_1)
- new net: J423. (Pin_1), J481. (Pin_1)
- new net: J516. (Pin_1), J546. (Pin_1)
- new net: J514. (Pin_1), J548. (Pin_1)
- new net: J350. (Pin_1), J396. (Pin_1)
- new net: J415. (Pin_1), J489. (Pin_1)
- new net: J527. (Pin_1), J536. (Pin_1)
- new net: J599. (Pin_1), J631. (Pin_1)
- new net: J427. (Pin_1), J477. (Pin_1)
- new net: J499. (Pin_1), J563. (Pin_1)
- new net: J424. (Pin_1), J480. (Pin_1)
- new net: J581. (Pin_1), J613. (Pin_1)
- new net: J517. (Pin_1), J545. (Pin_1)
- new net: J418. (Pin_1), J486. (Pin_1)
- new net: J573. (Pin_1), J605. (Pin_1)
- new net: J444. (Pin_1), J461. (Pin_1)
- new net: J372. (Pin_1), J375. (Pin_1)
- new net: J419. (Pin_1), J485. (Pin_1)
- new net: J366. (Pin_1), J381. (Pin_1)
- new net: J452. (Pin_1), J453. (Pin_1)
- new net: J447. (Pin_1), J458. (Pin_1)
- new net: J434. (Pin_1), J470. (Pin_1)
- new net: J582. (Pin_1), J614. (Pin_1)
- new net: J426. (Pin_1), J478. (Pin_1)
- new net: J530. (Pin_1), J533. (Pin_1)
- new net: J578. (Pin_1), J610. (Pin_1)
- new net: J501. (Pin_1), J561. (Pin_1)
- new net: J435. (Pin_1), J469. (Pin_1)
- new net: J503. (Pin_1), J559. (Pin_1)
- new net: J507. (Pin_1), J555. (Pin_1)
- new net: J353. (Pin_1), J393. (Pin_1)
- new net: J343. (Pin_1), J399. (Pin_1)
- new net: J414. (Pin_1), J490. (Pin_1)
- new net: J342. (Pin_1), J400. (Pin_1)
- new net: J437. (Pin_1), J467. (Pin_1)
- new net: J370. (Pin_1), J377. (Pin_1)
- new net: J373. (Pin_1), J374. (Pin_1)
- new net: J422. (Pin_1), J482. (Pin_1)
- new net: J526. (Pin_1), J537. (Pin_1)
- new net: J590. (Pin_1), J622. (Pin_1)
- new net: J367. (Pin_1), J380. (Pin_1)
- new net: J524. (Pin_1), J539. (Pin_1)
- new net: J579. (Pin_1), J611. (Pin_1)
- new net: J164. (Pin_1), J341. (Pin_1)
- new net: J580. (Pin_1), J612. (Pin_1)
- new net: J255. (Pin_1), J309. (Pin_1)
- new net: J362. (Pin_1), J385. (Pin_1)
- no-connect marks 47 -> 51
Other:
- note added: "*Looking at the car from behind"
- note added: "13-PIN MOLEX CONNECTOR"
- note added: "2103124-4"
- note added: "28-PIN OEM CONNECTOR"
- note added: "35"
- note added: "36"
- note added: "37"
- note added: "38"
- note added: "39"
- note added: "40"
- note added: "40-PIN MOLEX CONNECTOR"
- note added: "41"
- note added: "42"
- note added: "43"
- note added: "44"
- note added: "45"
- note added: "46"
- note added: "47"
- note added: "48"
- note added: "48-PIN OEM CONNECTOR"
- note added: "A"
- note added: "ATHP042P08EL16-H1"
- note added: "Accum"
- note added: "B"
- note added: "BS-01_M"
- note added: "BS-05_M"
- note added: "BS-09_M"
- note added: "C"
- note added: "CANaMon 1"
- note added: "CANaMon 2"
- note added: "CANaMon 3"
- note added: "CANaMon 4"
- note added: "CANaMon 5"
- note added: "CANaMon 6"
- note added: "CANaMon 7"
- note added: "CANaMon 8"
- note added: "CANaMon 9"
- note added: "CEN (CAN)"
- note added: "CEN (GND)"
- note added: "CEN, Resolver, RS232"
- note added: "DAISY CHAIN"
- note added: "DCDC (12V)"
- note added: "DCDC (HV)"
- note added: "ELRA2A0310"
- note added: "Energy Meter"
- note added: "GND_SENSE_F"
- note added: "GND_SENSE_R"
- note added: "HIP (12V)"
- note added: "HIP (HV)"
- note added: "HPK CONN"
- note added: "LV BAT"
- note added: "MOLEX CONNECTOR"
- note added: "PUMPS"
- note added: "RS232"
- note added: "Resolver"
- note removed: "BLUE"
- note removed: "GND_SENSE"

Commit message: accum stuff for connector pin out
thinking of calling this file "NU25_MCHA_Systems"
Parts:
- added BT1, BT2, BT3, BT4, BT5, BT6, BT7, BT8, BT9: Battery, symbol Device:Battery
- added J713, J714, J715, J716, J717, J718, J719, J720, J721, J722, J723, J724, J725, J726, J727, J728, J729, J730, J731, J732: Conn_01x01_Pin, symbol Connector:Conn_01x01_Pin
Connections:
- new net: BT9.2 (-), J732. (Pin_1)
- new net: BT7.2 (-), J729. (Pin_1)
- new net: BT7.1 (+), J726. (Pin_1)
- new net: BT2.1 (+), J717. (Pin_1)
- new net: BT2.2 (-), J719. (Pin_1)
- new net: BT3.2 (-), J721. (Pin_1)
- new net: BT1.1 (+), J715. (Pin_1)
- new net: BT1.2 (-), J716. (Pin_1)
- new net: BT3.1 (+), J718. (Pin_1)
- new net: BT6.1 (+), J724. (Pin_1)
- new net: BT8.1 (+), J728. (Pin_1)
- new net: BT6.2 (-), J727. (Pin_1)
- new net: BT4.1 (+), J720. (Pin_1)
- new net: BT9.1 (+), J730. (Pin_1)
- new net: BT8.2 (-), J731. (Pin_1)
- new net: BT5.1 (+), J722. (Pin_1)
- new net: BT5.2 (-), J725. (Pin_1)
Other:
- note added: "Dash"
- note added: "LVD/Precharge"
- note added: "NEG"
- note added: "POS"
- note added: "Pedal Box"
- note added: "Segment 1"
- note added: "Segment 2"
- note added: "Segment 3"
- note added: "Segment 4"
- note added: "Segment 5"
- note added: "Segment 6"
- note added: "Segment 7"
- note added: "Segment 8"
- note added: "Segment 9"
- note removed: "AIR +ve"

Commit message: accum wiring mostly done
need to add in fan banks (simplified version)
Parts:
- removed J1, J2: Conn_01x01_Pin, symbol Connector:Conn_01x01_Pin
- added 500V,100A: Fuse, symbol Device:Fuse
- added D1: Indicator Light, symbol Device:LED
- added J1, J2: Radlok, symbol Connector_Generic:Conn_01x01
- added J733, J734, J735, J736, J737, J738, J739, J740, J741, J742, J743, J744, J745, J746, J747, J748: Conn_01x01_Pin, symbol Connector:Conn_01x01_Pin
- added K1: IR +, symbol Relay:Relay_SPST-NO
- added K2: IR -, symbol Relay:Relay_SPST-NO
- added SW1: MSD, symbol Switch:SW_DPST_x2
Connections:
- net at J637. (Pin_1): now also J641. (Pin_1)
- net at J646. (Pin_1): now also J662. (Pin_1)
- net at J695. (Pin_1): now also J190. (Pin_1), J236. (Pin_1), J651. (Pin_1), J709. (Pin_1), K2.A2
- net at J723. (Pin_1): now also BT4.2 (-)
- net at J700. (Pin_1): now also J656. (Pin_1)
- net at J679. (Pin_1): now also J705. (Pin_1)
- net at J655. (Pin_1): now also J699. (Pin_1)
- net at J645. (Pin_1): now also J661. (Pin_1)
- net at J676. (Pin_1): now also J706. (Pin_1)
- net at J702. (Pin_1): now also J658. (Pin_1)
- net at J671. (Pin_1): now also J707. (Pin_1)
- net at J708. (Pin_1): now also J670. (Pin_1)
- net at J657. (Pin_1): now also J701. (Pin_1)
- net at J703. (Pin_1): now also J689. (Pin_1)
- net at J668. (Pin_1): now also J688. (Pin_1), J704. (Pin_1)
- net at J696. (Pin_1): now also J652. (Pin_1)
- net at J258. (Pin_1): now also J739. (Pin_1)
- net at J644. (Pin_1): now also J660. (Pin_1)
- net at J636. (Pin_1): now also J640. (Pin_1)
- net at J714. (Pin_1): now also 500V,100A.2, J2.1 (Pin_1)
- net at J713. (Pin_1): now also J1.1 (Pin_1), J746. (Pin_1), K1.13
- net at J642. (Pin_1): now also J638. (Pin_1)
- net at J635. (Pin_1): now also J639. (Pin_1)
- net at J3. (Pin_1): now also J733. (Pin_1), J738. (Pin_1), J741. (Pin_1), K1.14
- net at J257. (Pin_1): now also J742. (Pin_1), SW1.1 (A)
- net at J653. (Pin_1): now also J697. (Pin_1), J747. (Pin_1), K1.A2
- net at J710. (Pin_1): now also K2.A1
- net at J694. (Pin_1): now also J650. (Pin_1)
- net at J643. (Pin_1): now also J659. (Pin_1)
- net at J255. (Pin_1), J309. (Pin_1): now also SW1.2 (B)
- new net: J734. (Pin_1), J737. (Pin_1), J740. (Pin_1), K2.14
- new net: D1.2 (A), J735. (Pin_1)
- new net: J748. (Pin_1), K1.A1
- new net: D1.1 (K), J736. (Pin_1)
- new net: 500V,100A.1, K2.13
- no-connect marks 51 -> 83
Other:
- note added: "AIL"
- note added: "Accum +"
- note added: "HV"
- note added: "High Voltage Distribution"
- note added: "MOST NEG"
- note added: "MOST POS"
- note added: "Motor Controller"
- note added: "NEG IR"
- note added: "POS IR"
- note added: "Precharge/IRs"
- note added: "TS +"
- note added: "TS -"
- note added: "TS Stack"
- note removed: "AIR -ve"
- note removed: "IRs"
- note removed: "LVD/Precharge"
- moved on the sheet: BT1, BT2, BT3, BT4, BT5, BT6, BT7, BT8, BT9
