File: NU25 Connector Pinout/PCB/NU25 Connector Pinout/NU25 Connector Pinout.kicad_sch (KiCad schematic)
At the start: 762 parts, among them J1 Radlok, J10 Conn_01x01_Pin, J100 Conn_01x01_Pin, J101 Conn_01x01_Pin, J102 Conn_01x01_Pin, J103 Conn_01x01_Pin, J104 Conn_01x01_Pin, J105 Conn_01x01_Pin, J106 Conn_01x01_Pin, J107 Conn_01x01_Pin, J108 Conn_01x01_Pin, J109 Conn_01x01_Pin, J11 Conn_01x01_Pin, J110 Conn_01x01_Pin, J111 Conn_01x01_Pin, J112 Conn_01x01_Pin, J113 Conn_01x01_Pin, J114 Conn_01x01_Pin, J115 Conn_01x01_Pin, J116 Conn_01x01_Pin, J117 Conn_01x01_Pin, J118 Conn_01x01_Pin, J119 Conn_01x01_Pin, J12 Conn_01x01_Pin, J120 Conn_01x01_Pin, J121 Conn_01x01_Pin, J122 Conn_01x01_Pin, J123 Conn_01x01_Pin, J124 Conn_01x01_Pin, J125 Conn_01x01_Pin, J126 Conn_01x01_Pin, J127 Conn_01x01_Pin, J128 Conn_01x01_Pin, J129 Conn_01x01_Pin, J13 Conn_01x01_Pin, J130 Conn_01x01_Pin, J131 Conn_01x01_Pin, J132 Conn_01x01_Pin, J133 Conn_01x01_Pin, J134 Conn_01x01_Pin, J135 Conn_01x01_Pin, J136 Conn_01x01_Pin, J137 Conn_01x01_Pin, J138 Conn_01x01_Pin, J139 Conn_01x01_Pin, J14 Conn_01x01_Pin, J140 Conn_01x01_Pin, J141 Conn_01x01_Pin, J142 Conn_01x01_Pin, J143 Conn_01x01_Pin, J144 Conn_01x01_Pin, J145 Conn_01x01_Pin, J146 Conn_01x01_Pin, J147 Conn_01x01_Pin, J148 Conn_01x01_Pin, J149 Conn_01x01_Pin, J15 Conn_01x01_Pin, J150 Conn_01x01_Pin, J151 Conn_01x01_Pin, J152 Conn_01x01_Pin, J153 Conn_01x01_Pin, J154 Conn_01x01_Pin, J155 Conn_01x01_Pin, J156 Conn_01x01_Pin, J157 Conn_01x01_Pin, J158 Conn_01x01_Pin, J159 Conn_01x01_Pin, J16 Conn_01x01_Pin, J160 Conn_01x01_Pin, J161 Conn_01x01_Pin, J162 Conn_01x01_Pin, J163 Conn_01x01_Pin, J164 Conn_01x01_Pin, J165 Conn_01x01_Pin, J166 Conn_01x01_Pin, J167 Conn_01x01_Pin, J168 Conn_01x01_Pin, J169 Conn_01x01_Pin, J17 Conn_01x01_Pin, J170 Conn_01x01_Pin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

Commit message: nu25 electrical overview
motor controller pin out
estops
shutdown circuit breaks
Parts:
- removed SW1: MSD, symbol Switch:SW_DPST_x2
- added D2: MotorTempSens, symbol Device:D_TemperatureDependent
- added J749, J750: Conn_01x15_Pin, symbol Connector:Conn_01x15_Pin
- added J751, J753, J754: Conn_01x10_Pin, symbol Connector:Conn_01x10_Pin
- added J752: Conn_01x06_Pin, symbol Connector:Conn_01x06_Pin
- added J755, J756, J757, J758, J759, J760, J761, J762, J763, J764, J765, J766, J767, J768, J769: Conn_01x01_Pin, symbol Connector:Conn_01x01_Pin
- added SW1: Precharge, symbol Switch:SW_DIP_x01
- added SW10: E-STOP_DASH, symbol Switch:SW_Push_Open_Dual
- added SW2: Program Enable Switch, symbol Switch:SW_DPST_x2
- added SW4: E-STOP_TOP_RIGHT, symbol Switch:SW_Push_Open_Dual
- added SW5: E-STOP_TOP_LEFT, symbol Switch:SW_Push_Open_Dual
- added SW6: MSD_Interlock, symbol Switch:SW_DIP_x01
- added SW7: Brake-Over-Travel-Switch, symbol Switch:SW_DIP_x01
- added SW8: Inertia Switch, symbol Switch:SW_DIP_x01
- added SW9: TSMS, symbol Switch:SW_DIP_x01
Connections:
- net at J204. (Pin_1): now also J264. (Pin_1)
- net at J271. (Pin_1): now also J769. (Pin_1)
- net at J200. (Pin_1): now also J272. (Pin_1)
- net at J275. (Pin_1): now also J768. (Pin_1)
- net at J203. (Pin_1): now also J260. (Pin_1)
- net at J262. (Pin_1): now also D2.1 (K)
- net at J270. (Pin_1): now also D2.2 (A)
- net at J257. (Pin_1), J742. (Pin_1): now also SW6.1
- net at J255. (Pin_1), J309. (Pin_1): now also SW6.2
- net at J303. (Pin_1): now also J198. (Pin_1)
- net at J290. (Pin_1): now also J756. (Pin_1)
- net at J279. (Pin_1): now also J767. (Pin_1)
- net at J197. (Pin_1): now also J305. (Pin_1)
- net at J304. (Pin_1): now also J201. (Pin_1)
- net at J286. (Pin_1): now also J757. (Pin_1)
- net GND: now reaches J283. (Pin_1)
- net at J288. (Pin_1): now also SW2.2 (B)
- net at J259. (Pin_1): now also J764. (Pin_1)
- net at J306. (Pin_1): now also J202. (Pin_1)
- net Pullup?: now reaches J297. (Pin_1)
- net at J267. (Pin_1): now also J766. (Pin_1)
- net at J282. (Pin_1): now also J759. (Pin_1), SW2.1 (A)
- net at J263. (Pin_1): now also J765. (Pin_1)
- no-connect marks 83 -> 122
Other:
- note added: "*Refer to CM200 Hardware(HW) User Manual for pinout explanation - seach online for it"
- note added: "*Used for diagnostics and external PCBs"
- note added: "BSPD Breakout"
- note added: "CANaMons*"
- note added: "CEN*"
- note added: "DB 9 CONNECTOR"
- note added: "DEN*"
- note added: "E-Stop_Top_Left"
- note added: "E-Stop_Top_Right"
- note added: "HFR Breakout"
- note added: "HIP*"
- note added: "LEGEND"
- note added: "LVD*"
- note added: "PEN*"
- note added: "Precharge*"
- note added: "Service Handle"
- note added: "TSAL_Discharge Breakout"
- note added: "cos +ve"
- note added: "cos -ve"
- note added: "excitn otpt"
- note added: "excitn rtrn"
- note added: "sine +ve"
- note added: "sine -ve"
- note removed: "E-Stop_Left"
- note removed: "E-Stop_Right"
- note removed: "Precharge"
- title: NU25 Connector Pinout -> NU25 Electrical System Overview
- moved on the sheet: 500V,100A, BT1, BT2, BT3, BT4, BT5, BT6, BT7, BT8, BT9
