File: ELECTRICAL SYSTEM OVERVIEW/NU25 Electrical System Overview/NU25 Electrical System Overview.kicad_sch (KiCad schematic)
At the start: 792 parts, among them J1 Radlok, J10 Conn_01x01_Pin, J100 Conn_01x01_Pin, J101 Conn_01x01_Pin, J102 Conn_01x01_Pin, J103 Conn_01x01_Pin, J104 Conn_01x01_Pin, J105 Conn_01x01_Pin, J106 Conn_01x01_Pin, J107 Conn_01x01_Pin, J108 Conn_01x01_Pin, J109 Conn_01x01_Pin, J11 Conn_01x01_Pin, J110 Conn_01x01_Pin, J111 Conn_01x01_Pin, J112 Conn_01x01_Pin, J113 Conn_01x01_Pin, J114 Conn_01x01_Pin, J115 Conn_01x01_Pin, J116 Conn_01x01_Pin, J117 Conn_01x01_Pin, J118 Conn_01x01_Pin, J119 Conn_01x01_Pin, J12 Conn_01x01_Pin, J120 Conn_01x01_Pin, J121 Conn_01x01_Pin, J122 Conn_01x01_Pin, J123 Conn_01x01_Pin, J124 Conn_01x01_Pin, J125 Conn_01x01_Pin, J126 Conn_01x01_Pin, J127 Conn_01x01_Pin, J128 Conn_01x01_Pin, J129 Conn_01x01_Pin, J13 Conn_01x01_Pin, J130 Conn_01x01_Pin, J131 Conn_01x01_Pin, J132 Conn_01x01_Pin, J133 Conn_01x01_Pin, J134 Conn_01x01_Pin, J135 Conn_01x01_Pin, J136 Conn_01x01_Pin, J137 Conn_01x01_Pin, J138 Conn_01x01_Pin, J139 Conn_01x01_Pin, J14 Conn_01x01_Pin, J140 Conn_01x01_Pin, J141 Conn_01x01_Pin, J142 Conn_01x01_Pin, J143 Conn_01x01_Pin, J144 Conn_01x01_Pin, J145 Conn_01x01_Pin, J146 Conn_01x01_Pin, J147 Conn_01x01_Pin, J148 Conn_01x01_Pin, J149 Conn_01x01_Pin, J15 Conn_01x01_Pin, J150 Conn_01x01_Pin, J151 Conn_01x01_Pin, J152 Conn_01x01_Pin, J153 Conn_01x01_Pin, J154 Conn_01x01_Pin, J155 Conn_01x01_Pin, J156 Conn_01x01_Pin, J157 Conn_01x01_Pin, J158 Conn_01x01_Pin, J159 Conn_01x01_Pin, J16 Conn_01x01_Pin, J160 Conn_01x01_Pin, J161 Conn_01x01_Pin, J162 Conn_01x01_Pin, J163 Conn_01x01_Pin, J164 Conn_01x01_Pin, J165 Conn_01x01_Pin, J166 Conn_01x01_Pin, J167 Conn_01x01_Pin, J168 Conn_01x01_Pin, J169 Conn_01x01_Pin, J17 Conn_01x01_Pin, J170 Conn_01x01_Pin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

Commit message: remaining of nu25 connector pinout to nu25 electrical system overview
Parts:
- added J770, J771, J772, J773, J774, J775, J776, J777: Conn_01x01_Pin, symbol Connector:Conn_01x01_Pin
- added SW3: GLVMS, symbol Switch:SW_DIP_x01
Connections:
- no-connect marks 122 -> 123
Other:
- note added: "*generates I_CEN"
- note added: "*generates I_PACK"
- note added: "Current Sensor"
- note added: "MOLEX CONN"
- note added: "OEM CONNECTOR"
